File: pa1010d-breakout.kicad_pcb (KiCad board)
At the start: 2 copper layers, 21 x 24 mm, 10 parts, among them J1 Conn_01x05_Male, J2 Conn_01x05_Male, U1 PA1010D

Commit message: refactor: change pin layout for easier trace routing. close #4
Parts:
- C1, C2: moved to F.Cu
- moved C1 13.4 mm to (106.2, 90.4)
- moved C2 11.7 mm to (106.2, 92.7)
Connections:
- J1 pad 1: /SDA -> /TX
- J1 pad 2: /SCL -> /RX
- J1 pad 4: /TX -> /SCL
- J1 pad 5: /RX -> /SDA
- J2 pad 1: /VBACKUP -> /NRESET
- J2 pad 2: +3V3 -> GND
- J2 pad 4: GND -> /VBACKUP
- J2 pad 5: /NRESET -> +3V3
Routing:
- net +3V3: track 18.7 -> 11.0 mm
- net /WAKEUP: track 18.6 -> 12.3 mm
- net GND: track 6.88 -> 12.7 mm, vias 2 -> 4
- net /VBACKUP: track 14.6 -> 8.87 mm
- net /TX: track 10.4 -> 5.33 mm
- net /RX: track 13.6 -> 9.00 mm
- net /1PPS: track 15.8 -> 11.7 mm
- net /SDA: track 16.9 -> 20.1 mm
- net /SCL: track 17.0 -> 15.2 mm

Commit message: refactor: add pull up / down resistors
Co-authored-by: Chinmay Pendharkar <notthetup@gmail.com>
Parts:
- added R1: 10k, Passives:R_0805_2012Metric_Pad1.15x1.40mm_HandSolder, B.Cu at (107.7, 76.7)
- added R2: 10k, Passives:R_0805_2012Metric_Pad1.15x1.40mm_HandSolder, B.Cu at (99.3, 77.7)
- renumbered C2 to C1, C1 to C2
Connections:
- J1 pad 1: /TX -> /RX
- J1 pad 2: /RX -> /TX
- U1 pad 4: /RX -> /TX
- U1 pad 5: /TX -> /RX
Routing:
- net +3V3: track 11.0 -> 31.2 mm
- net GND: track 12.7 -> 31.2 mm, vias 4 -> 0
- net /NRESET: track 17.7 -> 25.4 mm
- net /TX: track 5.33 -> 9.00 mm
- net /SDA: track 20.1 -> 18.3 mm
- net /RX: track 9.00 -> 10.2 mm
- net /SCL: track 15.2 -> 14.6 mm
- removed copper zone on B.Cu, net GND
Other:
- board text added: "RST"
